Commit message: feat: integrate multi-robot SLAM, autonomous exploration, and dockerized simulation
This commit introduces the core mapping and autonomous navigation architecture for the multi-robot swarm, alongside crucial physics fixes for Gazebo Harmonic.

### New Features & Architecture
- Dockerized Workflow: Added Dockerfile and docker-compose.yml to isolate simulation, mapping, and navigation.
- Swarm SLAM Package: Created swarm_slam with launch and config files for SLAM Toolbox and Nav2.
- Autonomous Exploration: Integrated m-explore-ros2 and tuned explore.yaml.
- Automated Mapping: Added auto_mapping.launch.py to bring up the full stack.

### Simulation & Physics Fixes (swarm_simulation)
- Fix diff-drive kinematics scale: Replaced <wheel_diameter> with <wheel_radius> to fix the 16.5% velocity scaling bug.
- DART physics solver stability: Converted wheel collisions to sphere and forced frictionless casters.
- Prevent chassis dragging & tipping: Shrunk base_link collision box, shifted CM to stop wheelies, and added front caster.
- Soften spawn impact: Lowered spawn Z-height to 0.01m in launch script.

### Perception
- Updated swarm_perception dependencies.

File: multi_robot_qr_nav/swarm_simulation/urdf/tb3_namespaced.urdf.xacro (robot description, xacro)
@@ -34,12 +34,20 @@
     <collision>
       <origin xyz="-0.064 0 0.047" rpy="0 0 0"/>
-      <geometry><box size="0.266 0.266 0.094"/></geometry>
+      <geometry><box size="0.266 0.266 0.050"/></geometry>
     </collision>
     <inertial>
-      <origin xyz="0 0 0" rpy="0 0 0"/>
+      <origin xyz="-0.064 0 0" rpy="0 0 0"/>
       <mass value="1.3729096e+00"/>
       <inertia ixx="8.7002718e-03" ixy="-4.7576583e-05" ixz="1.1160499e-04" iyy="8.6195418e-03" iyz="-3.5422299e-06" izz="1.4612727e-02" />
     </inertial>
   </link>
+  <gazebo reference="${prefix}base_link">
+    <mu1>0.0</mu1>
+    <mu2>0.0</mu2>
+    <kp>1000000.0</kp>
+    <kd>100.0</kd>
+    <minDepth>0.001</minDepth>
+    <maxVel>1.0</maxVel>
+  </gazebo>
   <!-- Left Wheel -->
   <joint name="${prefix}wheel_left_joint" type="continuous">
@@ -48,4 +56,5 @@
     <origin xyz="0.0 0.144 0.023" rpy="-1.57 0 0"/>
     <axis xyz="0 0 1"/>
+    <dynamics damping="0.0" friction="0.0"/>
   </joint>
   <link name="${prefix}wheel_left_link">
@@ -59,5 +68,5 @@
     <collision>
       <origin xyz="0 0 0" rpy="0 0 0"/>
-      <geometry><cylinder length="0.018" radius="0.033"/></geometry>
+      <geometry><sphere radius="0.033"/></geometry>
     </collision>
     <inertial>
@@ -67,4 +76,12 @@
     </inertial>
   </link>
+  <gazebo reference="${prefix}wheel_left_link">
+    <mu1>1.0</mu1>
+    <mu2>1.0</mu2>
+    <kp>1000000.0</kp>
+    <kd>100.0</kd>
+    <minDepth>0.001</minDepth>
+    <maxVel>0.1</maxVel>
+  </gazebo>
   <!-- Right Wheel -->
   <joint name="${prefix}wheel_right_joint" type="continuous">
@@ -73,4 +90,5 @@
     <origin xyz="0.0 -0.144 0.023" rpy="-1.57 0 0"/>
     <axis xyz="0 0 1"/>
+    <dynamics damping="0.0" friction="0.0"/>
   </joint>
   <link name="${prefix}wheel_right_link">
@@ -84,5 +102,5 @@
     <collision>
       <origin xyz="0 0 0" rpy="0 0 0"/>
-      <geometry><cylinder length="0.018" radius="0.033"/></geometry>
+      <geometry><sphere radius="0.033"/></geometry>
     </collision>
     <inertial>
@@ -92,23 +110,76 @@
     </inertial>
   </link>
+  <gazebo reference="${prefix}wheel_right_link">
+    <mu1>1.0</mu1>
+    <mu2>1.0</mu2>
+    <kp>1000000.0</kp>
+    <kd>100.0</kd>
+    <minDepth>0.001</minDepth>
+    <maxVel>0.1</maxVel>
+  </gazebo>
   <!-- Casters -->
   <joint name="${prefix}caster_back_right_joint" type="fixed">
     <parent link="${prefix}base_link"/>
     <child link="${prefix}caster_back_right_link"/>
-    <origin xyz="-0.177 -0.064 -0.004" rpy="-1.57 0 0"/>
+    <origin xyz="-0.177 -0.064 -0.004" rpy="0 0 0"/>
+    <dynamics damping="0.0" friction="0.0"/>
   </joint>
   <link name="${prefix}caster_back_right_link">
-    <collision><origin xyz="0 0.001 0" rpy="0 0 0"/><geometry><box size="0.030 0.009 0.020"/></geometry></collision>
+    <collision>
+      <origin xyz="0 0 0.027" rpy="0 0 0"/>
+      <geometry><sphere radius="0.033"/></geometry>
+    </collision>
     <inertial><mass value="0.005"/><inertia ixx="0.001" ixy="0.0" ixz="0.0" iyy="0.001" iyz="0.0" izz="0.001"/></inertial>
   </link>
+  <gazebo reference="${prefix}caster_back_right_link">
+    <mu1>0.0</mu1>
+    <mu2>0.0</mu2>
+    <kp>1000000.0</kp>
+    <kd>100.0</kd>
+    <minDepth>0.001</minDepth>
+    <maxVel>1.0</maxVel>
+  </gazebo>
   <joint name="${prefix}caster_back_left_joint" type="fixed">
     <parent link="${prefix}base_link"/>
     <child link="${prefix}caster_back_left_link"/>
-    <origin xyz="-0.177 0.064 -0.004" rpy="-1.57 0 0"/>
+    <origin xyz="-0.177 0.064 -0.004" rpy="0 0 0"/>
+    <dynamics damping="0.0" friction="0.0"/>
   </joint>
   <link name="${prefix}caster_back_left_link">
-    <collision><origin xyz="0 0.001 0" rpy="0 0 0"/><geometry><box size="0.030 0.009 0.020"/></geometry></collision>
+    <collision>
+      <origin xyz="0 0 0.027" rpy="0 0 0"/>
+      <geometry><sphere radius="0.033"/></geometry>
+    </collision>
     <inertial><mass value="0.005"/><inertia ixx="0.001" ixy="0.0" ixz="0.0" iyy="0.001" iyz="0.0" izz="0.001"/></inertial>
   </link>
+  <gazebo reference="${prefix}caster_back_left_link">
+    <mu1>0.0</mu1>
+    <mu2>0.0</mu2>
+    <kp>1000000.0</kp>
+    <kd>100.0</kd>
+    <minDepth>0.001</minDepth>
+    <maxVel>1.0</maxVel>
+  </gazebo>
+  <!-- Front Caster (Added for Anti-Tip Stability) -->
+  <joint name="${prefix}caster_front_joint" type="fixed">
+    <parent link="${prefix}base_link"/>
+    <child link="${prefix}caster_front_link"/>
+    <origin xyz="0.06 0 -0.004" rpy="0 0 0"/>
+  </joint>
+  <link name="${prefix}caster_front_link">
+    <collision>
+      <origin xyz="0 0 0.027" rpy="0 0 0"/>
+      <geometry><sphere radius="0.033"/></geometry>
+    </collision>
+    <inertial><mass value="0.005"/><inertia ixx="0.001" ixy="0.0" ixz="0.0" iyy="0.001" iyz="0.0" izz="0.001"/></inertial>
+  </link>
+  <gazebo reference="${prefix}caster_front_link">
+    <mu1>0.0</mu1>
+    <mu2>0.0</mu2>
+    <kp>1000000.0</kp>
+    <kd>100.0</kd>
+    <minDepth>0.001</minDepth>
+    <maxVel>1.0</maxVel>
+  </gazebo>
   <!-- IMU -->
   <joint name="${prefix}imu_joint" type="fixed">
@@ -176,9 +247,9 @@
       <right_joint>${prefix}wheel_right_joint</right_joint>
       <wheel_separation>0.287</wheel_separation>
-      <wheel_diameter>0.066</wheel_diameter>
-      <max_linear_acceleration>1.0</max_linear_acceleration>
-      <min_linear_acceleration>-1.0</min_linear_acceleration>
-      <max_angular_acceleration>2.0</max_angular_acceleration>
-      <min_angular_acceleration>-2.0</min_angular_acceleration>
+      <wheel_radius>0.033</wheel_radius>
+      <max_linear_acceleration>2.0</max_linear_acceleration>
+      <min_linear_acceleration>-2.0</min_linear_acceleration>
+      <max_angular_acceleration>4.0</max_angular_acceleration>
+      <min_angular_acceleration>-4.0</min_angular_acceleration>
       <topic>/${robot_name}/cmd_vel</topic>
       <odom_topic>/${robot_name}/odom</odom_topic>
@@ -186,4 +257,5 @@
       <frame_id>${prefix}odom</frame_id>
       <child_frame_id>${prefix}base_footprint</child_frame_id>
+      <odom_publish_frequency>30</odom_publish_frequency>
     </plugin>
   </gazebo>

Commit message: Tune Nav2 and explore-lite for optimal mapping and QR scanning - Adjusted LiDAR and Costmap ranges to a balanced 4.0m to force the robot to drive deep into rooms and sweep walls closely for QR detection, rather than mapping from afar. - Increased physical LiDAR resolution to 1440 samples to prevent beam spreading and ensure solid map grid generation without speckled gaps. - Tuned Regulated Pure Pursuit parameters (lookahead_dist: 0.3) to prevent the robot from cutting corners and triggering false collision aborts. - Adjusted inflation_radius (0.35) and cost_scaling_factor (2.0) to force the global planner to route safely down the center of corridors. - Disabled  to prevent the robot from freezing out of fear in narrow hallways. - Lowered explore-lite  to 0.25 to encourage mapping deeper into corners before considering a room complete.

File: multi_robot_qr_nav/swarm_simulation/urdf/tb3_namespaced.urdf.xacro (robot description, xacro)
@@ -122,5 +122,5 @@
     <parent link="${prefix}base_link"/>
     <child link="${prefix}caster_back_right_link"/>
-    <origin xyz="-0.177 -0.064 -0.004" rpy="0 0 0"/>
+    <origin xyz="-0.177 -0.064 -0.002" rpy="0 0 0"/>
     <dynamics damping="0.0" friction="0.0"/>
   </joint>
@@ -143,5 +143,5 @@
     <parent link="${prefix}base_link"/>
     <child link="${prefix}caster_back_left_link"/>
-    <origin xyz="-0.177 0.064 -0.004" rpy="0 0 0"/>
+    <origin xyz="-0.177 0.064 -0.002" rpy="0 0 0"/>
     <dynamics damping="0.0" friction="0.0"/>
   </joint>
@@ -165,5 +165,5 @@
     <parent link="${prefix}base_link"/>
     <child link="${prefix}caster_front_link"/>
-    <origin xyz="0.06 0 -0.004" rpy="0 0 0"/>
+    <origin xyz="0.06 0 -0.002" rpy="0 0 0"/>
   </joint>
   <link name="${prefix}caster_front_link">
@@ -272,5 +272,5 @@
         <scan>
           <horizontal>
-            <samples>360</samples>
+            <samples>1440</samples>
             <resolution>1</resolution>
             <min_angle>0.0</min_angle>
@@ -278,5 +278,5 @@
           </horizontal>
         </scan>
-        <range><min>0.120</min><max>3.5</max><resolution>0.015</resolution></range>
+        <range><min>0.120</min><max>4.0</max><resolution>0.015</resolution></range>
       </ray>
     </sensor>
